Commit message: URDF: measure from CAD, add meshes
Rebuild rover_description from the SolidWorks assembly (Assem1.STEP)
instead of estimates. Wheel size, track, wheelbase, body extents and
the LiDAR/camera/IMU poses all come from the CAD; each link gets an
STL visual mesh exported in its own frame.

- tools/step_to_meshes.py regenerates the meshes from the STEP file
- LiDAR yaw = pi (A1 driver 0 deg faces the motor tail, which is at the
  rear) and IMU yaw = -pi/2 (GY-521 pin row faces the rear); both still
  need confirming on hardware
- Un-ignore the URDF meshes (*.stl was ignored for OpenSCAD exports)
  and mark STL as binary

Co-Authored-By: Claude Opus 5.5 <noreply@anthropic.com>

File: ros/rover_description/urdf/rover.urdf.xacro (robot description, xacro)
@@ -4,53 +4,65 @@
   Frames (REP-103: +X forward, +Y left, +Z up):
     base_footprint            on the ground, directly under base_link
-    `- base_link             centre of the four axles, at axle height
-        +- chassis           (visual/collision only, fixed)
+    `- base_link              centre of the four axles, at axle height
+        +- chassis            the tub (visual/collision only, fixed)
         +- front_left_wheel  \
         +- front_right_wheel | continuous joints, spin about +Y
         +- rear_left_wheel   |
         +- rear_right_wheel  /
-        +- laser
-        +- imu_link
-        `- camera_link
+        +- laser              RPLIDAR A1M8 scan centre
+        +- imu_link           MPU6050 chip
+        `- camera_link        Pi Camera lens, front face
             `- camera_link_optical   (+Z forward, +X right, +Y down)
+  Every dimension below is measured from the SolidWorks assembly
+  (CAD Files/Old Prototype Design/Assem1.STEP), which is the robot as built.
+  The visual meshes in meshes/ come from the same file through
+  tools/step_to_meshes.py; if the CAD changes, re-run that AND update the
+  numbers here. The two must agree.
   The electronics (Pi, ESP32, L298N, battery) are not modelled - they are part
-  of the chassis.
-  Values marked MEASURE are estimates from the CAD render. Everything in this
-  file is a property at the top, so measuring the robot only means editing
-  numbers here. All lengths in metres, angles in radians.
+  of the chassis. All lengths in metres, angles in radians.
 -->
 <robot name="guide_dog_rover" xmlns:xacro="http://www.ros.org/wiki/xacro">
   <!-- ================================================================== -->
-  <!-- Measured                                                            -->
-  <!-- ================================================================== -->
-  <xacro:property name="wheel_radius"   value="0.055"/>  <!-- 11 cm diameter -->
-  <xacro:property name="track_width"    value="0.240"/>  <!-- L wheel centre to R wheel centre -->
-  <!-- ================================================================== -->
-  <!-- MEASURE - estimates from the CAD                                    -->
-  <!-- ================================================================== -->
-  <xacro:property name="wheel_width"    value="0.045"/>  <!-- tyre tread width -->
-  <xacro:property name="wheelbase"      value="0.140"/>  <!-- front axle to rear axle -->
-  <!-- Chassis tub: outer dimensions, and where its underside sits relative
-       to the axle line (negative = below the axles). -->
-  <xacro:property name="chassis_length" value="0.280"/>
-  <xacro:property name="chassis_width"  value="0.180"/>  <!-- must be < track_width - wheel_width -->
-  <xacro:property name="chassis_height" value="0.130"/>
-  <xacro:property name="chassis_bottom" value="-0.020"/>
-  <!-- Sensor poses relative to base_link: x forward, y left, z up. -->
-  <xacro:property name="laser_x"  value="0.080"/>
-  <xacro:property name="laser_y"  value="0.000"/>
-  <xacro:property name="laser_z"  value="0.150"/>
-  <xacro:property name="laser_yaw" value="0.0"/>        <!-- 0 = the LiDAR's 0 deg faces forward; pi if mounted backwards -->
-  <xacro:property name="imu_x"    value="0.000"/>
-  <xacro:property name="imu_y"    value="0.000"/>
-  <xacro:property name="imu_z"    value="0.020"/>
-  <!-- Rotation that takes the robot frame onto the IMU board's printed axes.
-       Board X->forward, Y->left, Z->up means all zero. -->
+  <!-- Drivetrain                                                          -->
+  <!-- ================================================================== -->
+  <xacro:property name="wheel_radius"   value="0.0598"/>  <!-- 119.6 mm tyre -->
+  <xacro:property name="wheel_width"    value="0.041"/>
+  <xacro:property name="track_width"    value="0.2146"/>  <!-- L wheel centre to R wheel centre -->
+  <xacro:property name="wheelbase"      value="0.1473"/>  <!-- front axle to rear axle -->
+  <!-- ================================================================== -->
+  <!-- Chassis tub: outer bounding box, relative to base_link              -->
+  <!-- ================================================================== -->
+  <xacro:property name="chassis_length" value="0.2743"/>
+  <xacro:property name="chassis_width"  value="0.2083"/>
+  <xacro:property name="chassis_height" value="0.1296"/>
+  <xacro:property name="chassis_bottom" value="-0.0153"/>  <!-- underside is 15 mm below the axles -->
+  <!-- ================================================================== -->
+  <!-- Sensors: pose relative to base_link (x forward, y left, z up)       -->
+  <!-- ================================================================== -->
+  <!-- RPLIDAR A1M8. Origin is the spin axis at the height of the laser
+       emitter/receiver, i.e. the scan plane - not the bottom of the unit.
+       laser_yaw = pi because the driver's 0 deg points toward the motor
+       (the A1's narrow tail), and the tail faces the rear. Verify with the
+       box test: an object straight ahead must appear at +X in RViz. -->
+  <xacro:property name="laser_x"   value="0.08805"/>
+  <xacro:property name="laser_y"   value="-0.0011"/>
+  <xacro:property name="laser_z"   value="0.1730"/>
+  <xacro:property name="laser_yaw" value="${pi}"/>
+  <!-- MPU6050 on its GY-521 board, flat on the tub floor, pin header toward
+       the rear. On a GY-521 the printed +Y arrow points away from the pins and
+       +X runs along them, so the board's X faces the robot's right:
+       yaw = -pi/2. Verify with the tilt tests before trusting it. -->
+  <xacro:property name="imu_x"     value="-0.00455"/>
+  <xacro:property name="imu_y"     value="-0.0080"/>
+  <xacro:property name="imu_z"     value="-0.0097"/>
   <xacro:property name="imu_roll"  value="0.0"/>
   <xacro:property name="imu_pitch" value="0.0"/>
-  <xacro:property name="imu_yaw"   value="0.0"/>
-  <xacro:property name="camera_x"     value="0.140"/>
-  <xacro:property name="camera_y"     value="0.000"/>
-  <xacro:property name="camera_z"     value="0.120"/>
+  <xacro:property name="imu_yaw"   value="${-pi/2}"/>
+  <!-- Pi Camera, centre of the lens front, on the front face of the tub.
+       The CAD uses a Camera Module v2.1 model; the v3 actually fitted has the
+       same 25 x 24 mm board, so any lens offset is a few millimetres. -->
+  <xacro:property name="camera_x"     value="0.13975"/>
+  <xacro:property name="camera_y"     value="0.0"/>
+  <xacro:property name="camera_z"     value="0.0469"/>
   <xacro:property name="camera_pitch" value="0.0"/>     <!-- positive = tilted DOWN -->
   <!-- Masses, only used by simulators. -->
@@ -60,7 +72,7 @@
   <!-- Derived - do not edit                                               -->
   <!-- ================================================================== -->
-  <xacro:property name="PI" value="3.14159265358979"/>
   <xacro:property name="half_track" value="${track_width / 2}"/>
   <xacro:property name="half_base"  value="${wheelbase / 2}"/>
+  <xacro:property name="mesh_dir"   value="package://rover_description/meshes"/>
   <!-- ================================================================== -->
   <!-- Materials                                                           -->
@@ -68,11 +80,13 @@
   <material name="grey">  <color rgba="0.75 0.75 0.75 1"/></material>
   <material name="black"> <color rgba="0.10 0.10 0.10 1"/></material>
-  <material name="red">   <color rgba="0.85 0.15 0.15 1"/></material>
+  <material name="dark">  <color rgba="0.20 0.20 0.20 1"/></material>
+  <material name="green"> <color rgba="0.10 0.45 0.20 1"/></material>
   <material name="blue">  <color rgba="0.20 0.30 0.80 1"/></material>
   <!-- ================================================================== -->
   <!-- Inertia helpers                                                     -->
   <!-- ================================================================== -->
-  <xacro:macro name="box_inertia" params="m x y z">
+  <xacro:macro name="box_inertia" params="m x y z *origin">
     <inertial>
+      <xacro:insert_block name="origin"/>
       <mass value="${m}"/>
       <inertia ixx="${m*(y*y+z*z)/12}" ixy="0" ixz="0"
@@ -100,20 +114,23 @@
   </joint>
   <link name="base_link"/>
-  <!-- The tub is a separate link so base_link stays exactly on the axle
-       centre while the box sits where the real body is. -->
+  <!-- The chassis link shares base_link's origin so its mesh drops straight
+       in; the collision box is offset to where the tub actually is. -->
   <joint name="chassis_joint" type="fixed">
     <parent link="base_link"/>
     <child  link="chassis"/>
-    <origin xyz="0 0 ${chassis_bottom + chassis_height / 2}" rpy="0 0 0"/>
+    <origin xyz="0 0 0" rpy="0 0 0"/>
   </joint>
   <link name="chassis">
     <visual>
-      <geometry><box size="${chassis_length} ${chassis_width} ${chassis_height}"/></geometry>
+      <geometry><mesh filename="${mesh_dir}/chassis.stl"/></geometry>
       <material name="grey"/>
     </visual>
     <collision>
+      <origin xyz="0 0 ${chassis_bottom + chassis_height / 2}" rpy="0 0 0"/>
       <geometry><box size="${chassis_length} ${chassis_width} ${chassis_height}"/></geometry>
     </collision>
-    <xacro:box_inertia m="${chassis_mass}" x="${chassis_length}" y="${chassis_width}" z="${chassis_height}"/>
+    <xacro:box_inertia m="${chassis_mass}" x="${chassis_length}" y="${chassis_width}" z="${chassis_height}">
+      <origin xyz="0 0 ${chassis_bottom + chassis_height / 2}" rpy="0 0 0"/>
+    </xacro:box_inertia>
   </link>
   <!-- ================================================================== -->
@@ -134,10 +151,9 @@
     <link name="${prefix}_wheel">
       <visual>
-        <origin xyz="0 0 0" rpy="${PI/2} 0 0"/>
-        <geometry><cylinder radius="${wheel_radius}" length="${wheel_width}"/></geometry>
+        <geometry><mesh filename="${mesh_dir}/${prefix}_wheel.stl"/></geometry>
         <material name="black"/>
       </visual>
       <collision>
-        <origin xyz="0 0 0" rpy="${PI/2} 0 0"/>
+        <origin xyz="0 0 0" rpy="${pi/2} 0 0"/>
         <geometry><cylinder radius="${wheel_radius}" length="${wheel_width}"/></geometry>
       </collision>
@@ -159,9 +175,11 @@
   <link name="laser">
     <visual>
-      <geometry><cylinder radius="0.035" length="0.040"/></geometry>
-      <material name="red"/>
-    </visual>
+      <geometry><mesh filename="${mesh_dir}/lidar.stl"/></geometry>
+      <material name="dark"/>
+    </visual>
+    <!-- Unit plus its mount: 62 mm tall, top 9 mm above the scan plane. -->
     <collision>
-      <geometry><cylinder radius="0.035" length="0.040"/></geometry>
+      <origin xyz="0 0 -0.0221" rpy="0 0 0"/>
+      <geometry><cylinder radius="0.036" length="0.0626"/></geometry>
     </collision>
   </link>
@@ -176,5 +194,5 @@
   <link name="imu_link">
     <visual>
-      <geometry><box size="0.02 0.015 0.003"/></geometry>
+      <geometry><mesh filename="${mesh_dir}/imu.stl"/></geometry>
       <material name="blue"/>
     </visual>
@@ -190,6 +208,6 @@
   <link name="camera_link">
     <visual>
-      <geometry><box size="0.010 0.025 0.025"/></geometry>
-      <material name="black"/>
+      <geometry><mesh filename="${mesh_dir}/camera.stl"/></geometry>
+      <material name="green"/>
     </visual>
   </link>
@@ -199,5 +217,5 @@
     <parent link="camera_link"/>
     <child  link="camera_link_optical"/>
-    <origin xyz="0 0 0" rpy="${-PI/2} 0 ${-PI/2}"/>
+    <origin xyz="0 0 0" rpy="${-pi/2} 0 ${-pi/2}"/>
   </joint>
   <link name="camera_link_optical"/>

Commit message: Use measured wheels (110 mm) and track (240 mm) everywhere
The robot's wheels are 110 mm and its track 240 mm, measured. Set in all
three places that hold the geometry: the firmware (WHEEL_DIAMETER_M,
TRACK_WIDTH_M), wheel_odometry's defaults, and the URDF (wheel_radius
0.055, track_width 0.240; the CAD wheel mesh is scaled radially to match).
Sensor poses are unchanged. LiDAR now 0.23 m above the floor.

Supersedes the urdf-65mm-wheels branch. Firmware compiles (395 KB).

Co-Authored-By: Claude Opus 5.5 <noreply@anthropic.com>

File: ros/rover_description/urdf/rover.urdf.xacro (robot description, xacro)
@@ -15,5 +15,7 @@
             `- camera_link_optical   (+Z forward, +X right, +Y down)
   Every dimension below is measured from the SolidWorks assembly
-  (CAD Files/Old Prototype Design/Assem1.STEP), which is the robot as built.
+  (CAD Files/Old Prototype Design/Assem1.STEP), which is the robot as built -
+  except the wheels and track, measured on the robot: 110 mm wheels (CAD 119.6)
+  and a 240 mm track (CAD 214.6).
   The visual meshes in meshes/ come from the same file through
   tools/step_to_meshes.py; if the CAD changes, re-run that AND update the
@@ -26,7 +28,12 @@
   <!-- Drivetrain                                                          -->
   <!-- ================================================================== -->
-  <xacro:property name="wheel_radius"   value="0.0598"/>  <!-- 119.6 mm tyre -->
+  <!-- Wheel size and track are measured on the robot, not taken from the CAD
+       (119.6 mm tyres, 214.6 mm track). The axles are fixed to the body, so
+       every sensor pose below stays as measured from the CAD. The CAD wheel
+       mesh is scaled radially to match; its tread width is left as is. -->
+  <xacro:property name="wheel_radius"   value="0.055"/>   <!-- 110 mm wheel, measured -->
   <xacro:property name="wheel_width"    value="0.041"/>
-  <xacro:property name="track_width"    value="0.2146"/>  <!-- L wheel centre to R wheel centre -->
+  <xacro:property name="cad_wheel_radius" value="0.0598"/>  <!-- size of meshes/*_wheel.stl -->
+  <xacro:property name="track_width"    value="0.240"/>   <!-- L wheel centre to R wheel centre, measured -->
   <xacro:property name="wheelbase"      value="0.1473"/>  <!-- front axle to rear axle -->
   <!-- ================================================================== -->
@@ -151,5 +158,7 @@
     <link name="${prefix}_wheel">
       <visual>
-        <geometry><mesh filename="${mesh_dir}/${prefix}_wheel.stl"/></geometry>
+        <!-- Mesh axle is along Y: scale X and Z (the diameter), keep Y (the width). -->
+        <geometry><mesh filename="${mesh_dir}/${prefix}_wheel.stl"
+                        scale="${wheel_radius / cad_wheel_radius} 1 ${wheel_radius / cad_wheel_radius}"/></geometry>
         <material name="black"/>
       </visual>

Commit message: Shaft extender with built-in encoder disc, sensor holder, 290 mm track
encoder_extender.py (CadQuery) builds:
- Shaft extender: slides over the motor's 6 mm round shaft (bore 6.3,
  two M1.7 set screws), carries a 32-slot encoder disc 5 mm off the
  motor face, and gives the wheel a new 6 mm shaft (15 mm, with a flat
  for its set screw) 25 mm further out. Prints standing on the disc,
  no supports.
- Encoder holder: clamps round the gearbox (37 mm default, measure),
  shelf with fences and an adjustable M3 slot puts the LM393 fork
  around the disc with the beam across the slot ring.
Clash-checked against motor, sensor and wheel proxies: no overlaps.

Moving each wheel out 25 mm widens the track: 0.240 -> 0.290 in the
firmware, Pi odometry and URDF. The new disc gives 32 ticks per wheel
turn (was 140 with the old disc); marked to confirm with encoder_test.
Firmware compiles.

Co-Authored-By: Claude Opus 5.5 <noreply@anthropic.com>

File: ros/rover_description/urdf/rover.urdf.xacro (robot description, xacro)
@@ -17,5 +17,6 @@
   (CAD Files/Old Prototype Design/Assem1.STEP), which is the robot as built -
   except the wheels and track, measured on the robot: 110 mm wheels (CAD 119.6)
-  and a 240 mm track (CAD 214.6).
+  and a 240 mm track on the bare motor shafts (CAD 214.6), now 290 mm with the
+  25 mm shaft extenders that make room for the encoders (encoder_extender.py).
   The visual meshes in meshes/ come from the same file through
   tools/step_to_meshes.py; if the CAD changes, re-run that AND update the
@@ -35,5 +36,5 @@
   <xacro:property name="wheel_width"    value="0.041"/>
   <xacro:property name="cad_wheel_radius" value="0.0598"/>  <!-- size of meshes/*_wheel.stl -->
-  <xacro:property name="track_width"    value="0.240"/>   <!-- L wheel centre to R wheel centre, measured -->
+  <xacro:property name="track_width"    value="0.290"/>   <!-- L wheel centre to R wheel centre: 240 + 2 x 25 extender -->
   <xacro:property name="wheelbase"      value="0.1473"/>  <!-- front axle to rear axle -->
   <!-- ================================================================== -->
